File: elec/BusinessCardV1/Accelerometer_Circle_Setup.kicad_sch (KiCad schematic)
At the start: 18 parts, among them U12 SN74LVC08APWR, U13 SN74LVC08APWR, U18 ADXL327BCPZ, U4 TLV8544DR, U5 TLV8544DR, U6 TC4069UBFTEL_N

Commit message: Circle wiring
Parts:
- added R21, R22: 0, symbol Device:R
- added U19: TLV8544DR, D14_TEX, symbol TLV8544DR:TLV8544DR
- added U7: TC4069UBFTEL_N, TSSOP14_TOS, symbol TC4069UBFTELN:TC4069UBFTEL_N
Connections:
- net Blue_LED is gone; now on net op_y3: U6.5
- net Green_LED is gone; now on net op_y4: U6.9
- net OutFirst is gone; now on net ~{y2}: U6.4
- net Power3V3 is gone; now on net RingPower: U6.14
- net Red_LED is gone; now on net op_y5: U6.11
- net Reset is gone; now on net op_y6: U6.13
- net ~{Blue_LED} is gone; now on net ~{y3}: U6.6
- net ~{Green_LED} is gone; now on net ~{y4}: U6.8
- net ~{Red_LED} is gone; now on net ~{y5}: U6.10
- net ~{Reset} is gone; now on net ~{y6}: U6.12
- net ADXL_X_OUT: now also U19.3 (+INA)
- net GND: now also R22.2, U19.11 (V), U7.7
- net RingPower: now also R21.1, U19.4 (V+), U7.14
- net ~{y1}: now reaches U12.1 (1A)
- net ~{y1}: now also U6.2
- net op_y4: now reaches U12.10 (3B)
- net op_y4: now also U5.14 (OUTD)
- net Y5: now reaches U12.11 (4Y)
- net ~{y4}: now reaches U12.12 (4A)
- net op_y5: now reaches U12.13 (4B)
- net op_y5: now also U4.1 (OUTA)
- net op_y2: now reaches U12.2 (1B)
- net op_y2: now also U5.7 (OUTB), U6.3
- net Y2: now reaches U12.3 (1Y)
- net ~{y2}: now reaches U12.4 (2A)
- net op_y3: now reaches U12.5 (2B)
- net op_y3: now also U5.8 (OUTC)
- net Y3: now reaches U12.6 (2Y)
- net Y4: now reaches U12.8 (3Y)
- net ~{y3}: now reaches U12.9 (3A)
- net Y1: now reaches U5.1 (OUTA), U6.1
- net ~{y5}: now reaches U13.1 (1A)
- net op_y8: now reaches U13.10 (3B)
- net op_y8: now also U4.14 (OUTD)
- net op_y6: now reaches U13.2 (1B)
- net op_y6: now also U4.7 (OUTB)
- net Y6: now reaches U13.3 (1Y)
- net ~{y6}: now reaches U13.4 (2A)
- net op_y7: now reaches U13.5 (2B)
- net op_y7: now also U4.8 (OUTC), U7.1
- net Y7: now reaches U13.6 (2Y)
- net Y8: now reaches U13.8 (3Y)
- net ~{y7}: now reaches U13.9 (3A)
- net ~{y7}: now also U7.2
- new net: R21.2, R22.1, U19.2 (INA)
- new net x: U19.1 (OUTA), U7.3
- new net ~{x}: U7.4
- no-connect marks 9 -> 20
Other:
- moved on the sheet: U12, U13
