File: elec/BusinessCardV1/Accelerometer_Circle_Setup.kicad_sch (KiCad schematic)
At the start: 22 parts, among them U12 SN74LVC08APWR, U13 SN74LVC08APWR, U18 ADXL327BCPZ, U19 TLV8544DR, U4 TLV8544DR, U5 TLV8544DR, U6 TC4069UBFTEL_N, U7 TC4069UBFTEL_N

Commit message: All footprint and start of PCB
Parts:
- R12, R13, R14, R15, R16, R17, R18, R19, R20, R21, R22: footprint (none) -> Resistor_SMD:R_0603_1608Metric_Pad0.98x0.95mm_HandSolder
- U18: footprint CP_16_5A_ADI -> ADXL327BCPZ:CP_16_5A_ADI
- U19, U4, U5: footprint D14_TEX -> TLV8544DR:D14_TEX
- U6, U7: footprint TSSOP14_TOS -> TC4069UBFTELN:TSSOP14_TOS
Changed lines of the file:
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@@
 			)
 		)
-		(property "Footprint" ""
+		(property "Footprint" "Resistor_SMD:R_0603_1608Metric_Pad0.98x0.95mm_HandSolder"
 			(at 55.88 88.138 90)
 			(effects
@@
 			)
 		)
-		(property "Footprint" ""
+		(property "Footprint" "Resistor_SMD:R_0603_1608Metric_Pad0.98x0.95mm_HandSolder"
 			(at 133.35 149.098 90)
 			(effects
@@
 			)
 		)
-		(property "Footprint" ""
+		(property "Footprint" "Resistor_SMD:R_0603_1608Metric_Pad0.98x0.95mm_HandSolder"
 			(at 78.74 88.138 90)
 			(effects
@@
 			)
 		)
-		(property "Footprint" ""
+		(property "Footprint" "Resistor_SMD:R_0603_1608Metric_Pad0.98x0.95mm_HandSolder"
 			(at 101.6 88.138 90)
 			(effects
@@
 			)
 		)
-		(property "Footprint" "D14_TEX"
+		(property "Footprint" "TLV8544DR:D14_TEX"
 			(at 127 170.18 0)
 			(effects
@@
 			)
 		)
-		(property "Footprint" ""
+		(property "Footprint" "Resistor_SMD:R_0603_1608Metric_Pad0.98x0.95mm_HandSolder"
 			(at 86.36 88.138 90)
 			(effects
@@
 			)
 		)
-		(property "Footprint" ""
+		(property "Footprint" "Resistor_SMD:R_0603_1608Metric_Pad0.98x0.95mm_HandSolder"
 			(at 48.26 88.138 90)
 			(effects
@@
 			)
 		)
-		(property "Footprint" "TSSOP14_TOS"
+		(property "Footprint" "TC4069UBFTELN:TSSOP14_TOS"
 			(at 83.7946 135.89 0)
 			(effects
@@
 			)
 		)
-		(property "Footprint" "CP_16_5A_ADI"
+		(property "Footprint" "ADXL327BCPZ:CP_16_5A_ADI"
 			(at 60.96 35.56 0)
 			(effects
@@
 			)
 		)
-		(property "Footprint" "TSSOP14_TOS"
+		(property "Footprint" "TC4069UBFTELN:TSSOP14_TOS"
 			(at 35.5346 135.89 0)
 			(effects
@@
 			)
 		)
-		(property "Footprint" ""
+		(property "Footprint" "Resistor_SMD:R_0603_1608Metric_Pad0.98x0.95mm_HandSolder"
 			(at 71.12 88.138 90)
 			(effects
@@
 			)
 		)
-		(property "Footprint" "D14_TEX"
+		(property "Footprint" "TLV8544DR:D14_TEX"
 			(at 27.94 100.33 0)
 			(effects
@@
 			)
 		)
-		(property "Footprint" ""
+		(property "Footprint" "Resistor_SMD:R_0603_1608Metric_Pad0.98x0.95mm_HandSolder"
 			(at 140.97 149.098 90)
 			(effects
@@
 			)
 		)
-		(property "Footprint" ""
+		(property "Footprint" "Resistor_SMD:R_0603_1608Metric_Pad0.98x0.95mm_HandSolder"
 			(at 93.98 88.138 90)
 			(effects
@@
 			)
 		)
-		(property "Footprint" ""
+		(property "Footprint" "Resistor_SMD:R_0603_1608Metric_Pad0.98x0.95mm_HandSolder"
 			(at 63.5 88.138 90)
 			(effects
@@
 			)
 		)
-		(property "Footprint" ""
+		(property "Footprint" "Resistor_SMD:R_0603_1608Metric_Pad0.98x0.95mm_HandSolder"
 			(at 109.22 88.138 90)
 			(effects
@@
 			)
 		)
-		(property "Footprint" "D14_TEX"
+		(property "Footprint" "TLV8544DR:D14_TEX"
 			(at 96.52 100.33 0)
 			(effects

Commit message: Started layout
Connections:
- no-connect marks 20 -> 29
Changed lines of the file:
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@@
+	)
+	(no_connect
+		(at 167.64 180.34)
+	)
+	(no_connect
+		(at 127 180.34)
 	)
 	(no_connect
@@
 	)
 	(no_connect
+		(at 127 182.88)
+	)
+	(no_connect
+		(at 167.64 175.26)
+	)
+	(no_connect
 		(at 77.47 179.07)
+	)
+	(no_connect
+		(at 167.64 185.42)
 	)
 	(no_connect
@@
 	)
 	(no_connect
+		(at 127 185.42)
+	)
+	(no_connect
 		(at 60.96 50.8)
+	)
+	(no_connect
+		(at 167.64 182.88)
 	)
 	(no_connect
@@
 	(no_connect
 		(at 116.84 43.18)
+	)
+	(no_connect
+		(at 167.64 170.18)
 	)
 	(no_connect
@@
 	)
 	(no_connect
+		(at 167.64 172.72)
+	)
+	(no_connect
