File: elec/BusinessCardV1/Accelerometer_Circle_LED.kicad_sch (KiCad schematic)
At the start: 0 parts

Commit message: heheheha
Parts:
- added D1, D10, D11, D12, D13, D14, D15, D16, D2, D3, D4, D5, D6, D7, D8, D9: QBLP595-R, FP-QBLP595-R-MFG, symbol QBLP595:QTB-LED-0002
- added R4: 680, symbol Device:R
- added U10, U11, U12, U13, U8, U9: SN74LVC08APWR, SN74LVC08APWR:SOP65P640X120-14N, symbol SN74LVC08APWR:SN74LVC08APWR
- added U4, U5: TLV8544DR, D14_TEX, symbol TLV8544DR:TLV8544DR
- added U6, U7: TC4069UBFTEL_N, TSSOP14_TOS, symbol TC4069UBFTELN:TC4069UBFTEL_N
Connections:
- new net: D16.2 (ANODE_(+)), U11.11 (4Y)
- new net: D13.2 (ANODE_(+)), U11.3 (1Y)
- new net: D14.2 (ANODE_(+)), U11.6 (2Y)
- new net: D15.2 (ANODE_(+)), U11.8 (3Y)
- new net: D1.1 (CATHODE_(-)), D10.1 (CATHODE_(-)), D11.1 (CATHODE_(-)), D12.1 (CATHODE_(-)), D13.1 (CATHODE_(-)), D14.1 (CATHODE_(-)), D15.1 (CATHODE_(-)), D16.1 (CATHODE_(-)), D2.1 (CATHODE_(-)), D3.1 (CATHODE_(-)), D4.1 (CATHODE_(-)), D5.1 (CATHODE_(-)), D6.1 (CATHODE_(-)), D7.1 (CATHODE_(-)), D8.1 (CATHODE_(-)), D9.1 (CATHODE_(-)), R4.2
- new net: D8.2 (ANODE_(+)), U9.11 (4Y)
- new net: D4.2 (ANODE_(+)), U8.11 (4Y)
- new net: D1.2 (ANODE_(+)), U8.3 (1Y)
- new net: D2.2 (ANODE_(+)), U8.6 (2Y)
- new net: D3.2 (ANODE_(+)), U8.8 (3Y)
- new net: D7.2 (ANODE_(+)), U9.8 (3Y)
- new net: D10.2 (ANODE_(+)), U10.6 (2Y)
- new net: D11.2 (ANODE_(+)), U10.8 (3Y)
- new net: D12.2 (ANODE_(+)), U10.11 (4Y)
- new net: D9.2 (ANODE_(+)), U10.3 (1Y)
- new net: D6.2 (ANODE_(+)), U9.6 (2Y)
- new net: D5.2 (ANODE_(+)), U9.3 (1Y)
- new net GND: R4.1, U10.7 (GND), U11.7 (GND), U12.7 (GND), U13.7 (GND), U4.11 (V), U5.11 (V), U8.7 (GND), U9.7 (GND)
- new net RingPower: U10.14 (VCC), U11.14 (VCC), U12.14 (VCC), U13.14 (VCC), U4.4 (V+), U5.4 (V+), U8.14 (VCC), U9.14 (VCC)
- new net not x: U10.1 (1A), U10.12 (4A), U10.4 (2A), U10.9 (3A), U11.1 (1A), U11.12 (4A), U11.4 (2A), U11.9 (3A)
- new net x: U8.1 (1A), U8.12 (4A), U8.4 (2A), U8.9 (3A), U9.1 (1A), U9.12 (4A), U9.4 (2A), U9.9 (3A)

Commit message: pew
Parts:
- removed U12, U13: SN74LVC08APWR, SN74LVC08APWR:SOP65P640X120-14N, symbol SN74LVC08APWR:SN74LVC08APWR
- removed U4, U5: TLV8544DR, D14_TEX, symbol TLV8544DR:TLV8544DR
- removed U6, U7: TC4069UBFTEL_N, TSSOP14_TOS, symbol TC4069UBFTELN:TC4069UBFTEL_N
Connections:
- net not x renamed ~{x}
Other:
- moved on the sheet: D13, D14, D15, D16, D5, D6, D7, D8, R4, U11, U9

Commit message: Circle wiring
Connections:
- net Y7: now reaches U11.10 (3B)
- net Y7: now also U9.10 (3B)
- net Y8: now reaches U11.13 (4B)
- net Y8: now also U9.13 (4B)
- net Y5: now reaches U11.2 (1B)
- net Y5: now also U9.2 (1B)
- net Y6: now reaches U11.5 (2B)
- net Y6: now also U9.5 (2B)
- net Y3: now reaches U8.10 (3B)
- net Y3: now also U10.10 (3B)
- net Y4: now reaches U8.13 (4B)
- net Y4: now also U10.13 (4B)
- net Y1: now reaches U8.2 (1B)
- net Y1: now also U10.2 (1B)
- net Y2: now reaches U8.5 (2B)
- net Y2: now also U10.5 (2B)
Other:
- moved on the sheet: D1, D10, D11, D12, D13, D14, D15, D16, D2, D3, D4, D5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

Commit message: All footprint and start of PCB
Parts:
- D1, D10, D11, D12, D13, D14, D15, D16, D2, D3, D4, D5, D6, D7, D8, D9: footprint FP-QBLP595-R-MFG -> LED_SMD:LED_0402_1005Metric_Pad0.77x0.64mm_HandSolder
- R4: footprint (none) -> Resistor_SMD:R_0603_1608Metric_Pad0.98x0.95mm_HandSolder
Changed lines of the file:
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@@
 			)
 		)
-		(property "Footprint" "FP-QBLP595-R-MFG"
+		(property "Footprint" "LED_SMD:LED_0402_1005Metric_Pad0.77x0.64mm_HandSolder"
 			(at 110.49 105.41 0)
 			(effects
@@
 			)
 		)
-		(property "Footprint" "FP-QBLP595-R-MFG"
+		(property "Footprint" "LED_SMD:LED_0402_1005Metric_Pad0.77x0.64mm_HandSolder"
 			(at 109.22 102.87 0)
 			(effects
@@
 			)
 		)
-		(property "Footprint" "FP-QBLP595-R-MFG"
+		(property "Footprint" "LED_SMD:LED_0402_1005Metric_Pad0.77x0.64mm_HandSolder"
 			(at 167.64 55.88 0)
 			(effects
@@
 			)
 		)
-		(property "Footprint" "FP-QBLP595-R-MFG"
+		(property "Footprint" "LED_SMD:LED_0402_1005Metric_Pad0.77x0.64mm_HandSolder"
 			(at 109.22 53.34 0)
 			(effects
@@
 			)
 		)
-		(property "Footprint" "FP-QBLP595-R-MFG"
+		(property "Footprint" "LED_SMD:LED_0402_1005Metric_Pad0.77x0.64mm_HandSolder"
 			(at 167.64 58.42 0)
 			(effects
@@
 			)
 		)
-		(property "Footprint" "FP-QBLP595-R-MFG"
+		(property "Footprint" "LED_SMD:LED_0402_1005Metric_Pad0.77x0.64mm_HandSolder"
 			(at 109.22 60.96 0)
 			(effects
@@
 			)
 		)
-		(property "Footprint" ""
+		(property "Footprint" "Resistor_SMD:R_0603_1608Metric_Pad0.98x0.95mm_HandSolder"
 			(at 106.68 141.478 90)
 			(effects
@@
 			)
 		)
-		(property "Footprint" "FP-QBLP595-R-MFG"
+		(property "Footprint" "LED_SMD:LED_0402_1005Metric_Pad0.77x0.64mm_HandSolder"
 			(at 167.64 100.33 0)
 			(effects
@@
 			)
 		)
-		(property "Footprint" "FP-QBLP595-R-MFG"
+		(property "Footprint" "LED_SMD:LED_0402_1005Metric_Pad0.77x0.64mm_HandSolder"
 			(at 167.64 60.96 0)
 			(effects
@@
 			)
 		)
-		(property "Footprint" "FP-QBLP595-R-MFG"
+		(property "Footprint" "LED_SMD:LED_0402_1005Metric_Pad0.77x0.64mm_HandSolder"
 			(at 167.64 105.41 0)
 			(effects
@@
 			)
 		)
-		(property "Footprint" "FP-QBLP595-R-MFG"
+		(property "Footprint" "LED_SMD:LED_0402_1005Metric_Pad0.77x0.64mm_HandSolder"
 			(at 109.22 100.33 0)
 			(effects
@@
 			)
 		)
-		(property "Footprint" "FP-QBLP595-R-MFG"
+		(property "Footprint" "LED_SMD:LED_0402_1005Metric_Pad0.77x0.64mm_HandSolder"
 			(at 167.64 97.79 0)
 			(effects
@@
 			)
 		)
-		(property "Footprint" "FP-QBLP595-R-MFG"
+		(property "Footprint" "LED_SMD:LED_0402_1005Metric_Pad0.77x0.64mm_HandSolder"
 			(at 109.22 55.88 0)
 			(effects
@@
 			)
 		)
-		(property "Footprint" "FP-QBLP595-R-MFG"
+		(property "Footprint" "LED_SMD:LED_0402_1005Metric_Pad0.77x0.64mm_HandSolder"
 			(at 109.22 97.79 0)
 			(effects
@@
 			)
 		)
-		(property "Footprint" "FP-QBLP595-R-MFG"
+		(property "Footprint" "LED_SMD:LED_0402_1005Metric_Pad0.77x0.64mm_HandSolder"
 			(at 167.64 53.34 0)
 			(effects
@@
 			)
 		)
-		(property "Footprint" "FP-QBLP595-R-MFG"
+		(property "Footprint" "LED_SMD:LED_0402_1005Metric_Pad0.77x0.64mm_HandSolder"
 			(at 167.64 102.87 0)
 			(effects
@@
 			)
 		)
-		(property "Footprint" "FP-QBLP595-R-MFG"
+		(property "Footprint" "LED_SMD:LED_0402_1005Metric_Pad0.77x0.64mm_HandSolder"
 			(at 109.22 58.42 0)
 			(effects

Commit message: PCB routed
Parts:
- added C17, C18, C19, C20: 1uf, CL10B105KP8NNNC:CAPC1608X90N, symbol CL10B105KP8NNNC:CL10B105KP8NNNC
Connections:
- net GND: now also C17.1, C18.1, C19.1, C20.1
- net RingPower: now also C17.2, C18.2, C19.2, C20.2
