File: elec/BusinessCardV1/Buttons.kicad_sch (KiCad schematic)
At the start: 0 parts

Commit message: Button working i guess i hope
Parts:
- added C15: 4.7uf, CL10B105KP8NNNC:CAPC1608X90N, symbol CL10B105KP8NNNC:CL10B105KP8NNNC
- added C16: 10uf, CL10B105KP8NNNC:CAPC1608X90N, symbol CL10B105KP8NNNC:CL10B105KP8NNNC
- added R34, R36: 0, symbol Device:R
- added R35: 42.2, symbol Device:R
- added U21: IQS228B00000000TSR, IQS228B00000000TSR:SOT95P280X100-6N, symbol IQS228B00000000TSR:IQS228B00000000TSR
Connections:
- new net: C15.1, R35.1, U21.5 (VDDHI)
- new net: R36.2, U21.3 (CTRL/ND)
- new net: R34.2, U21.1 (OUT)
- new net: C16.1, U21.4 (VREG)
- new net +3.3V: R35.2
- new net GND: C15.2, C16.2, U21.2 (GND)
- new net RingBTN: R34.1, R36.1
- new net TouchSensor: U21.6 (CX)

Commit message: All footprint and start of PCB
Parts:
- R34, R35, R36: footprint (none) -> Resistor_SMD:R_0603_1608Metric_Pad0.98x0.95mm_HandSolder
Changed lines of the file:
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@@
 			)
 		)
-		(property "Footprint" ""
+		(property "Footprint" "Resistor_SMD:R_0603_1608Metric_Pad0.98x0.95mm_HandSolder"
 			(at 114.808 33.02 90)
 			(effects
@@
 			)
 		)
-		(property "Footprint" ""
+		(property "Footprint" "Resistor_SMD:R_0603_1608Metric_Pad0.98x0.95mm_HandSolder"
 			(at 96.52 71.882 90)
 			(effects
@@
 			)
 		)
-		(property "Footprint" ""
+		(property "Footprint" "Resistor_SMD:R_0603_1608Metric_Pad0.98x0.95mm_HandSolder"
 			(at 123.19 55.372 90)
 			(effects

Commit message: PCB routed
Parts:
- added J4: 6130XX11121_61300211121, Header1x2:Header1x2_SMD, symbol Header1x2:6130XX11121_61300211121
- added R37: 0, Resistor_SMD:R_0603_1608Metric_Pad0.98x0.95mm_HandSolder, symbol Device:R
Connections:
- net GND: now also R37.1
- net TouchSensor: now also J4.1
- new net Pad: J4.2, R37.2
