File: elec/BusinessCardV1/Power.kicad_sch (KiCad schematic)
At the start: 18 parts, among them J1 61300411121, J2 6130XX11121_61300211121, Q1 DMG2305UX-7, Q2 DMG2305UX-7, U1 *, U14 MCP73831T-2DCI_OT, U2 SN74LVC2G74DCTR, U3 TPS7A0233DBVR

Commit message: Started layout
Parts:
- added J3: 6130XX11121_61300211121, Header1x2:Header1x2_SMD, symbol Header1x2:6130XX11121_61300211121
Connections:
- net +3.3V: now also J3.2
- net GND: now also J3.1

Commit message: Push before destroying everything
Connections:
- net +3.3V: no longer J3.2
- net V_Bat: now also J3.2
Changed lines of the file:
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@@
-	(wire
-		(pts
-			(xy 260.35 45.72) (xy 260.35 41.91)
-		)
-		(stroke
-			(width 0)
-			(type default)
-		)
-	)
 	(wire
 		(pts
@@
 	(label "SDO"
 		(at 48.26 54.61 0)
-		(effects
-			(font
-				(size 1.27 1.27)
-			)
-			(justify left bottom)
-		)
-	)
-	(label "Power3V3"
-		(at 260.35 41.91 0)
 		(effects
 			(font
@@
 		)
 	)
+	(label "V_Bat"
+		(at 247.65 121.92 0)
+		(effects
+			(font
+				(size 1.27 1.27)
+				(thickness 0.254)
+				(bold yes)
+			)
+			(justify left bottom)
+		)
+	)
 	(label "SDX"
 		(at 48.26 52.07 0)
@@
 			)
 			(justify left bottom)
+		)
+	)
+	(global_label "Power3V3"
+		(shape input)
+		(at 260.35 45.72 0)
+		(fields_autoplaced yes)
+		(effects
+			(font
+				(size 1.27 1.27)
+			)
+			(justify left)
+		)
+		(property "Intersheetrefs" "${INTERSHEET_REFS}"
+			(at 272.4671 45.72 0)
+			(effects
+				(font
+					(size 1.27 1.27)
+				)
+				(justify left)
+				(hide yes)
+			)
 		)
 	)
@@
 					(unit 1)
 				)
-			)
-		)
-	)
-	(symbol
-		(lib_id "power:+3.3V")
-		(at 247.65 121.92 0)
-		(unit 1)
-		(exclude_from_sim no)
-		(in_bom yes)
-		(on_board yes)
-		(dnp no)
-		(fields_autoplaced yes)
-		(property "Reference" "#PWR055"
-			(at 247.65 125.73 0)
-			(effects
-				(font
-					(size 1.27 1.27)
-				)
-				(hide yes)
-			)
-		)
-		(property "Value" "+3.3V"
-			(at 247.65 116.84 0)
-			(effects
-				(font
-					(size 1.27 1.27)
-				)
-			)
-		)
-		(property "Footprint" ""
-			(at 247.65 121.92 0)
-			(effects
-				(font
-					(size 1.27 1.27)
-				)
-				(hide yes)
-			)
-		)
-		(property "Datasheet" ""
-			(at 247.65 121.92 0)
-			(effects
-				(font
-					(size 1.27 1.27)
-				)
-				(hide yes)
-			)
-		)
-		(property "Description" "Power symbol creates a global label with name \"+3.3V\""
-			(at 247.65 121.92 0)
-			(effects
-				(font
-					(size 1.27 1.27)
-				)
-				(hide yes)
-			)
-		)
-		(pin "1"
-		)
-		(instances
-			(project "BusinessCardV1"
-				(path "/28a1e4b0-497b-455a-8c80-759850e7b173/9de3a60e-6635-4d18-85fa-31055f93e53d"
-					(reference "#PWR055")
-					(unit 1)
-				)

Commit message: PCB routed
Changed lines of the file:
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@@
 		)
 	)
+	(wire
+		(pts
+			(xy 95.25 72.39) (xy 95.25 69.85)
+		)
+		(stroke
+			(width 0)
+			(type default)
+		)
+	)
 	(polyline
 		(pts
@@
 	(wire
 		(pts
+			(xy 95.25 69.85) (xy 96.52 69.85)
+		)
+		(stroke
+			(width 0)
+			(type default)
+		)
+	)
+	(wire
+		(pts
 			(xy 252.73 45.72) (xy 260.35 45.72)
 		)
@@
 	(wire
 		(pts
+			(xy 96.52 72.39) (xy 95.25 72.39)
+		)
+		(stroke
+			(width 0)
+			(type default)
+		)
+	)
+	(wire
+		(pts
 			(xy 80.01 158.75) (xy 88.9 158.75)
 		)
@@
 	(symbol
 		(lib_id "power:GND")
-		(at 96.52 69.85 0)
+		(at 96.52 72.39 0)
 		(unit 1)
 		(exclude_from_sim no)
@@
 		(fields_autoplaced yes)
 		(property "Reference" "#PWR011"
-			(at 96.52 76.2 0)
+			(at 96.52 78.74 0)
 			(effects
 				(font
@@
 		)
 		(property "Value" "GND"
-			(at 96.52 74.93 0)
+			(at 96.52 77.47 0)
 			(effects
 				(font
@@
 		)
 		(property "Footprint" ""
-			(at 96.52 69.85 0)
+			(at 96.52 72.39 0)
 			(effects
 				(font
@@
 		)
 		(property "Datasheet" ""
-			(at 96.52 69.85 0)
+			(at 96.52 72.39 0)
 			(effects
 				(font
@@
 		)
 		(property "Description" "Power symbol creates a global label with name \"GND\" , ground"
-			(at 96.52 69.85 0)
+			(at 96.52 72.39 0)
 			(effects
 				(font
