File: elec/BusinessCardV1/RGB_LED_circuit.kicad_sch (KiCad schematic)
At the start: 38 parts, among them Q3 DMG2305UX-7, Q4 DMG2305UX-7, Q5 DMG2305UX-7, Q6 DMG1012UW-7, Q7 DMG1012UW-7, Q8 DMG1012UW-7, U15 TC4069UBFTEL_N, U16 SN74LVC1G139DCTR, U17 SN74LV161ADR, U20 TLC555CDR

Commit message: Easy part done, Glabel kind of worked
Connections:
- net Blue_LED: now also U16.7 (Y0); no longer U16.5 (Y2)
- net Red_LED: now also U16.5 (Y2); no longer U16.7 (Y0)

Commit message: PCB routed
Parts:
- added C21, C22, C23: 1uf, CL10B105KP8NNNC:CAPC1608X90N, symbol CL10B105KP8NNNC:CL10B105KP8NNNC
Connections:
- net GND: now also C21.1, C22.1, C23.1
- net Power3V3: now also C21.2, C22.2, C23.2
