File: elec/BusinessCardV1/BusinessCardV1.kicad_pcb (KiCad board)
At the start: 2 copper layers, 176.2 x 54 mm, 116 parts, among them J1 61300411121, J2 6130XX11121_61300211121, J3 6130XX11121_61300211121, J4 6130XX11121_61300211121, Q1 DMG2305UX-7, Q2 DMG2305UX-7, Q3 DMG2305UX-7, Q4 DMG2305UX-7, Q5 DMG2305UX-7, Q6 DMG1012UW-7, Q7 DMG1012UW-7, Q8 DMG1012UW-7, U1 *, U10 SN74LVC08APWR, U11 SN74LVC08APWR, U12 SN74LVC08APWR, U13 SN74LVC08APWR, U14 MCP73831T-2DCI_OT, U15 TC4069UBFTEL_N, U16 SN74LVC1G139DCTR, U17 SN74LV161ADR, U18 ADXL327BCPZ, U19 TLV8544DR, U2 SN74LVC2G74DCTR, U20 TLC555CDR, U21 IQS228B00000000TSR, U22 TPD12S520DBT, U3 TPS7A0233DBVR, U4 TLV8544DR, U5 TLV8544DR, U6 TC4069UBFTEL_N, U7 TC4069UBFTEL_N, U8 SN74LVC08APWR, U9 SN74LVC08APWR

Commit message: Gerber almost ready
Parts:
- added J5: 6130XX11121_61300211121, Header1x2:SMD_Header, F.Cu at (93.5, 78.5)
Routing:
- net V_Bat: track 43.7 -> 49.7 mm
Other:
- outline, holes or cut-outs redrawn
Changed lines of the file:
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@@
 			(outputformat 1)
 			(mirror no)
-			(drillshape 1)
+			(drillshape 0)
 			(scaleselection 1)
-			(outputdirectory "")
+			(outputdirectory "plot/")
 		)
 	)
@@
 		)
 	)
+	(footprint "Header1x2:SMD_Header"
+		(layer "F.Cu")
+		(at 93.54 78.54 90)
+		(property "Reference" "J5"
+			(at 0 -0.5 90)
+			(unlocked yes)
+			(layer "F.SilkS")
+			(hide yes)
+			(effects
+				(font
+					(size 1 1)
+					(thickness 0.1)
+				)
+			)
+		)
+		(property "Value" "6130XX11121_61300211121"
+			(at 0 1 90)
+			(unlocked yes)
+			(layer "F.Fab")
+			(hide yes)
+			(effects
+				(font
+					(size 1 1)
+					(thickness 0.15)
+				)
+			)
+		)
+		(property "Datasheet" ""
+			(at 0 0 90)
+			(unlocked yes)
+			(layer "F.Fab")
+			(hide yes)
+			(effects
+				(font
+					(size 1 1)
+					(thickness 0.15)
+				)
+			)
+		)
+		(property "Description" ""
+			(at 0 0 90)
+			(unlocked yes)
+			(layer "F.Fab")
+			(hide yes)
+			(effects
+				(font
+					(size 1 1)
+					(thickness 0.15)
+				)
+			)
+		)
+		(property "DigiKey_Part_Number" "732-5315-ND"
+			(at 0 0 90)
+			(unlocked yes)
+			(layer "F.Fab")
+			(hide yes)
+			(effects
+				(font
+					(size 1 1)
+					(thickness 0.15)
+				)
+			)
+		)
+		(property "SnapEDA_Link" "https://www.snapeda.com/parts/61300211121/Wurth+Electronics/view-part/?ref=snap"
+			(at 0 0 90)
+			(unlocked yes)
+			(layer "F.Fab")
+			(hide yes)
+			(effects
+				(font
+					(size 1 1)
+					(thickness 0.15)
+				)
+			)
+		)
+		(property "Description_1" "Connector Header Through Hole 2 position 0.100 (2.54mm)"
+			(at 0 0 90)
+			(unlocked yes)
+			(layer "F.Fab")
+			(hide yes)
+			(effects
+				(font
+					(size 1 1)
+					(thickness 0.15)
+				)
+			)
+		)
+		(property "MF" "Wurth Electronics"
+			(at 0 0 90)
+			(unlocked yes)
+			(layer "F.Fab")
+			(hide yes)
+			(effects
+				(font
+					(size 1 1)
+					(thickness 0.15)
+				)
+			)
+		)
+		(property "Package" "None"
+			(at 0 0 90)
+			(unlocked yes)
+			(layer "F.Fab")
+			(hide yes)
+			(effects
+				(font
+					(size 1 1)
+					(thickness 0.15)
+				)
+			)
+		)
+		(property "Check_prices" "https://www.snapeda.com/parts/61300211121/Wurth+Electronics/view-part/?ref=eda"
+			(at 0 0 90)
+			(unlocked yes)
+			(layer "F.Fab")
+			(hide yes)
+			(effects
+				(font
+					(size 1 1)
+					(thickness 0.15)
+				)
+			)
+		)
+		(property "MP" "61300211121"
+			(at 0 0 90)
+			(unlocked yes)
+			(layer "F.Fab")
+			(hide yes)
+			(effects
+				(font
+					(size 1 1)
+					(thickness 0.15)
+				)
+			)
+		)
+		(sheetname "/")
+		(sheetfile "BusinessCardV1.kicad_sch")
+		(attr through_hole)
+		(pad "1" smd roundrect
+			(at 0 0 90)
+			(size 8 2.3)
+			(layers "F.Cu" "F.Mask" "F.Paste")
+			(roundrect_rratio 0.08)
+			(net 2 "V_Bat")
+			(pintype "passive")
+		)
+		(embedded_fonts no)
+	)
 	(footprint "Resistor_SMD:R_0603_1608Metric_Pad0.98x0.95mm_HandSolder"
 		(layer "F.Cu")
@@
 		(layer "Dwgs.User")
 	)
-	(gr_rect
-		(start 92.5 82.6)
-		(end 94.5 82.6)
-		(stroke
-			(width 0.1)
-			(type default)
-		)
-		(fill no)
-		(layer "Dwgs.User")
-	)
 	(gr_line
 		(start 184.81 113.04)
@@
 		(layer "Dwgs.User")
 	)
+	(gr_arc
+		(start 94.75 74.54)
+		(mid 93.474288 95.017989)
+		(end 92.301058 74.533873)
+		(stroke
+			(width 0.05)
+			(type default)
+		)
+		(layer "Edge.Cuts")
+	)
+	(gr_line
+		(start 92.301058 82.62)
+		(end 94.75 82.63)
+		(stroke
+			(width 0.05)
+			(type default)
+		)
+		(layer "Edge.Cuts")
+	)
 	(gr_rect
 		(start 106.1 71.5)
@@
 		(layer "Edge.Cuts")
 	)
+	(gr_line
+		(start 94.75 74.54)
+		(end 94.75 82.63)
+		(stroke
+			(width 0.05)
+			(type default)
+		)
+		(layer "Edge.Cuts")
+	)
 	(gr_rect
 		(start 20.5 71)
@@
 		(layer "Edge.Cuts")
 	)
-	(gr_arc
-		(start 93.5 74.5)
-		(mid 95.278308 94.826134)
-		(end 89.997418 75.1176)
+	(gr_line
+		(start 92.301058 74.533874)
+		(end 92.301058 82.62)
 		(stroke
 			(width 0.05)
-			(type solid)
+			(type default)
 		)
 		(layer "Edge.Cuts")
@@
 	(segment
 		(start 79.936 72.676)
-		(end 96.921689 72.676)
+		(end 93.11 72.676)
 		(width 0.381)
 		(layer "F.Cu")
@@
 	)
 	(segment
+		(start 93.11 72.676)
+		(end 96.921689 72.676)
+		(width 0.381)
+		(layer "F.Cu")
+		(net 2)
+	)
+	(segment
 		(start 79.682 75.234)
 		(end 79.682 72.93)
@@
 	)
 	(segment
+		(start 93.54 73.106)
+		(end 93.11 72.676)
+		(width 0.381)
+		(layer "F.Cu")
+		(net 2)
+	)
+	(segment
 		(start 75.89 75.3102)
 		(end 75.89 79.6125)
 		(width 0.381)
 		(layer "F.Cu")
+		(net 2)
+	)
+	(segment
+		(start 93.54 78.54)
+		(end 93.54 73.106)
+		(width 0.381)
+		(layer "F.Cu")
