File: elec/BusinessCardV1/BusinessCardV1.kicad_pcb (KiCad board)
At the start: 2 copper layers, 176.2 x 54 mm, 117 parts, among them J1 61300411121, J2 6130XX11121_61300211121, J3 6130XX11121_61300211121, J4 6130XX11121_61300211121, J5 6130XX11121_61300211121, Q1 DMG2305UX-7, Q2 DMG2305UX-7, Q3 DMG2305UX-7, Q4 DMG2305UX-7, Q5 DMG2305UX-7, Q6 DMG1012UW-7, Q7 DMG1012UW-7, Q8 DMG1012UW-7, U1 *, U10 SN74LVC08APWR, U11 SN74LVC08APWR, U12 SN74LVC08APWR, U13 SN74LVC08APWR, U14 MCP73831T-2DCI_OT, U15 TC4069UBFTEL_N, U16 SN74LVC1G139DCTR, U17 SN74LV161ADR, U18 ADXL327BCPZ, U19 TLV8544DR, U2 SN74LVC2G74DCTR, U20 TLC555CDR, U21 IQS228B00000000TSR, U22 TPD12S520DBT, U3 TPS7A0233DBVR, U4 TLV8544DR, U5 TLV8544DR, U6 TC4069UBFTEL_N, U7 TC4069UBFTEL_N, U8 SN74LVC08APWR, U9 SN74LVC08APWR

Commit message: Everything is good
Other:
- outline, holes or cut-outs redrawn
- board text added: "CSB"
- board text added: "SCX"
- board text added: "SD0"
- board text added: "SDX"
- board text added: "V_Bat"
Changed lines of the file:
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@@
 		(embedded_fonts no)
 	)
+	(footprint "Header1x2:SMD_Header"
+		(layer "F.Cu")
+		(at 93.53 78.5 90)
+		(property "Reference" "J5"
+			(at 0 -0.5 90)
+			(unlocked yes)
+			(layer "F.SilkS")
+			(hide yes)
+			(effects
+				(font
+					(size 1 1)
+					(thickness 0.1)
+				)
+			)
+		)
+		(property "Value" "6130XX11121_61300211121"
+			(at 0 1 90)
+			(unlocked yes)
+			(layer "F.Fab")
+			(hide yes)
+			(effects
+				(font
+					(size 1 1)
+					(thickness 0.15)
+				)
+			)
+		)
+		(property "Datasheet" ""
+			(at 0 0 90)
+			(unlocked yes)
+			(layer "F.Fab")
+			(hide yes)
+			(effects
+				(font
+					(size 1 1)
+					(thickness 0.15)
+				)
+			)
+		)
+		(property "Description" ""
+			(at 0 0 90)
+			(unlocked yes)
+			(layer "F.Fab")
+			(hide yes)
+			(effects
+				(font
+					(size 1 1)
+					(thickness 0.15)
+				)
+			)
+		)
+		(property "DigiKey_Part_Number" "732-5315-ND"
+			(at 0 0 90)
+			(unlocked yes)
+			(layer "F.Fab")
+			(hide yes)
+			(effects
+				(font
+					(size 1 1)
+					(thickness 0.15)
+				)
+			)
+		)
+		(property "SnapEDA_Link" "https://www.snapeda.com/parts/61300211121/Wurth+Electronics/view-part/?ref=snap"
+			(at 0 0 90)
+			(unlocked yes)
+			(layer "F.Fab")
+			(hide yes)
+			(effects
+				(font
+					(size 1 1)
+					(thickness 0.15)
+				)
+			)
+		)
+		(property "Description_1" "Connector Header Through Hole 2 position 0.100 (2.54mm)"
+			(at 0 0 90)
+			(unlocked yes)
+			(layer "F.Fab")
+			(hide yes)
+			(effects
+				(font
+					(size 1 1)
+					(thickness 0.15)
+				)
+			)
+		)
+		(property "MF" "Wurth Electronics"
+			(at 0 0 90)
+			(unlocked yes)
+			(layer "F.Fab")
+			(hide yes)
+			(effects
+				(font
+					(size 1 1)
+					(thickness 0.15)
+				)
+			)
+		)
+		(property "Package" "None"
+			(at 0 0 90)
+			(unlocked yes)
+			(layer "F.Fab")
+			(hide yes)
+			(effects
+				(font
+					(size 1 1)
+					(thickness 0.15)
+				)
+			)
+		)
+		(property "Check_prices" "https://www.snapeda.com/parts/61300211121/Wurth+Electronics/view-part/?ref=eda"
+			(at 0 0 90)
+			(unlocked yes)
+			(layer "F.Fab")
+			(hide yes)
+			(effects
+				(font
+					(size 1 1)
+					(thickness 0.15)
+				)
+			)
+		)
+		(property "MP" "61300211121"
+			(at 0 0 90)
+			(unlocked yes)
+			(layer "F.Fab")
+			(hide yes)
+			(effects
+				(font
+					(size 1 1)
+					(thickness 0.15)
+				)
+			)
+		)
+		(sheetname "/")
+		(sheetfile "BusinessCardV1.kicad_sch")
+		(attr through_hole)
+		(pad "1" smd roundrect
+			(at 0 0 90)
+			(size 8 2.3)
+			(layers "F.Cu")
+			(roundrect_rratio 0.08)
+			(net 2 "V_Bat")
+			(pintype "passive")
+		)
+		(embedded_fonts no)
+	)
 	(footprint "SN74LVC2G74DCTR:SOP65P400X130-8N"
 		(layer "F.Cu")
@@
 		(at 41.328 77.248 180)
 		(property "Reference" "Q5"
-			(at -0.13 -2.548 0)
+			(at -0.892 -2.352 0)
 			(layer "F.SilkS")
 			(effects
@@
 		)
 		(fp_text user "*"
-			(at -2.7178 -5.5118 180)
+			(at -3.425 -4.73 180)
 			(unlocked yes)
 			(layer "F.SilkS")
@@
 		(tags "LED handsolder")
 		(property "Reference" "D20"
-			(at 0 -1.17 90)
+			(at -0.048 2.25 90)
 			(layer "F.SilkS")
 			(effects
@@
 		(tags "LED handsolder")
 		(property "Reference" "D21"
-			(at 0 -1.17 0)
+			(at 0.006 1.712 0)
 			(layer "F.SilkS")
 			(effects
@@
 		)
 	)
-	(footprint "Header1x2:SMD_Header"
-		(layer "F.Cu")
-		(at 93.54 78.54 90)
-		(property "Reference" "J5"
-			(at 0 -0.5 90)
-			(unlocked yes)
-			(layer "F.SilkS")
-			(hide yes)
-			(effects
-				(font
-					(size 1 1)
-					(thickness 0.1)
-				)
-			)
-		)
-		(property "Value" "6130XX11121_61300211121"
-			(at 0 1 90)
-			(unlocked yes)
-			(layer "F.Fab")
-			(hide yes)
-			(effects
-				(font
-					(size 1 1)
-					(thickness 0.15)
-				)
-			)
-		)
-		(property "Datasheet" ""
-			(at 0 0 90)
-			(unlocked yes)
-			(layer "F.Fab")
-			(hide yes)
-			(effects
-				(font
-					(size 1 1)
-					(thickness 0.15)
-				)
-			)
-		)
-		(property "Description" ""
-			(at 0 0 90)
-			(unlocked yes)
-			(layer "F.Fab")
-			(hide yes)
-			(effects
-				(font
-					(size 1 1)
-					(thickness 0.15)
-				)
-			)
-		)
-		(property "DigiKey_Part_Number" "732-5315-ND"
-			(at 0 0 90)
-			(unlocked yes)
-			(layer "F.Fab")
-			(hide yes)
-			(effects
-				(font
-					(size 1 1)
-					(thickness 0.15)
-				)
-			)
-		)
-		(property "SnapEDA_Link" "https://www.snapeda.com/parts/61300211121/Wurth+Electronics/view-part/?ref=snap"
-			(at 0 0 90)
-			(unlocked yes)
-			(layer "F.Fab")
-			(hide yes)
-			(effects
-				(font
-					(size 1 1)
-					(thickness 0.15)
-				)
-			)
-		)
-		(property "Description_1" "Connector Header Through Hole 2 position 0.100 (2.54mm)"
-			(at 0 0 90)
-			(unlocked yes)
-			(layer "F.Fab")
-			(hide yes)
-			(effects
-				(font
-					(size 1 1)
-					(thickness 0.15)
-				)
-			)
-		)
-		(property "MF" "Wurth Electronics"
-			(at 0 0 90)
-			(unlocked yes)
-			(layer "F.Fab")
-			(hide yes)
-			(effects
-				(font
-					(size 1 1)
-					(thickness 0.15)
-				)
-			)
-		)
-		(property "Package" "None"
-			(at 0 0 90)
-			(unlocked yes)
-			(layer "F.Fab")
-			(hide yes)
-			(effects
-				(font
-					(size 1 1)
-					(thickness 0.15)
-				)
-			)
-		)
-		(property "Check_prices" "https://www.snapeda.com/parts/61300211121/Wurth+Electronics/view-part/?ref=eda"
-			(at 0 0 90)
-			(unlocked yes)
-			(layer "F.Fab")
-			(hide yes)
-			(effects
-				(font
-					(size 1 1)
-					(thickness 0.15)
-				)
-			)
-		)
-		(property "MP" "61300211121"
-			(at 0 0 90)
-			(unlocked yes)
-			(layer "F.Fab")
-			(hide yes)
-			(effects
-				(font
-					(size 1 1)
-					(thickness 0.15)
-				)
-			)
-		)
-		(sheetname "/")
-		(sheetfile "BusinessCardV1.kicad_sch")
-		(attr through_hole)
-		(pad "1" smd roundrect
-			(at 0 0 90)
-			(size 8 2.3)
-			(layers "F.Cu" "F.Mask" "F.Paste")
-			(roundrect_rratio 0.08)
-			(net 2 "V_Bat")
-			(pintype "passive")
-		)
-		(embedded_fonts no)
-	)
 	(footprint "Resistor_SMD:R_0603_1608Metric_Pad0.98x0.95mm_HandSolder"
 		(layer "F.Cu")
@@
 		(tags "LED handsolder")
 		(property "Reference" "D22"
-			(at 0 -1.17 90)
+			(at -0.068 -2.024 90)
 			(layer "F.SilkS")
 			(effects
@@
 		(tags "ADXL327BCPZ ")
 		(property "Reference" "U18"
-			(at 0 0 11.25)
+			(at -3.301132 -3.035904 11.25)
 			(unlocked yes)
 			(layer "F.SilkS")
@@
 		)
 		(fp_text user "*"
-			(at -3.18135 -3.4486 180)
+			(at -3.755 -2.765 180)
 			(unlocked yes)
 			(layer "F.SilkS")
@@
 	)
 	(gr_rect
-		(start 106.1 71.5)
-		(end 111.1 124.5)
+		(start 106.1 72.56)
+		(end 111.1 123.35)
 		(stroke
 			(width 0.05)
@@
 		(layer "Edge.Cuts")
 	)
+	(gr_text "SD0\n"
+		(at 67.59 75.71 90)
+		(layer "F.SilkS")
+		(effects
+			(font
+				(size 0.5 0.5)
+				(thickness 0.1)
+			)
+			(justify left bottom)
+		)
+	)
+	(gr_text "CSB"
+		(at 72.6 75.69 90)
+		(layer "F.SilkS")
+		(effects
+			(font
+				(size 0.5 0.5)
+				(thickness 0.1)
+			)
+			(justify left bottom)
+		)
+	)
 	(gr_text "GND"
 		(at 98.9 72.9 0)
@@
 				(thickness 0.1)
 			)
+			(justify left bottom)
+		)
+	)
+	(gr_text "V_Bat"
+		(at 89.99 74.03 0)
+		(layer "F.SilkS")
+		(effects
+			(font
+				(size 0.5 0.5)
+				(thickness 0.1)
+			)
+			(justify left bottom)
+		)
+	)
+	(gr_text "SDX"
+		(at 69.86 75.63 90)
+		(layer "F.SilkS")
+		(effects
+			(font
+				(size 0.5 0.5)
+				(thickness 0.1)
+			)
+			(justify left bottom)
+		)
+	)
+	(gr_text "SCX"
+		(at 71.13 75.67 90)
+		(layer "F.SilkS")
+		(effects
+			(font
+				(size 0.5 0.5)
+				(thickness 0.1)
+			)
